File: code/robot_wiring_design/robot_wiring_design.kicad_pcb (KiCad board)
At the start: 2 copper layers, 248.7 x 150.6 mm, 6 parts, among them J1 Conn_02x20_Counter_Clockwise

Commit message: add the final pcb update the bom with lesspriced lidar add the new model of the 3d robot design
Parts:
- removed the REF** at (56.4, 85.9)
- removed the REF** at (72.5, 85.8)
- removed mux1: multiplexer, Connector_PinHeader_2.54mm:PinHeader_2x12_P2.54mm_Vertical
- added J2: sg90, Connector_Wire:SolderWirePad_1x01_SMD_5x10mm, F.Cu at (174.8, 95.0)
- added J3: MUX LEFT, Connector_PinHeader_2.54mm:PinHeader_1x12_P2.54mm_Vertical, F.Cu at (117.7, 138.8)
- added J4: alim buck 5V pad, Connector_Wire:SolderWirePad_1x01_SMD_5x10mm, F.Cu at (92.0, 40.5)
- added J5: alim buck gnd pad, Connector_Wire:SolderWirePad_1x01_SMD_5x10mm, F.Cu at (83.0, 41.2)
- added J6: ampli, TerminalBlock:TerminalBlock_MaiXu_MX126-5.0-05P_1x05_P5.00mm, F.Cu at (52.7, 133.5)
- added J_LIDAR1: LD06, TerminalBlock:TerminalBlock_MaiXu_MX126-5.0-04P_1x04_P5.00mm, F.Cu at (64.2, 117.5)
- added REF**: MountingHole_2.5mm, MountingHole:MountingHole_2.5mm, F.Cu at (98.2, 89.5)
- added REF**: MountingHole_2.5mm, MountingHole:MountingHole_2.5mm, F.Cu at (24.3, 110.5)
- added REF**: MountingHole_2.5mm, MountingHole:MountingHole_2.5mm, F.Cu at (101.9, 59.4)
- added REF**: MountingHole_2.5mm, MountingHole:MountingHole_2.5mm, F.Cu at (109.7, 34.9)
- added REF**: MountingHole_2.5mm, MountingHole:MountingHole_2.5mm, F.Cu at (113.0, 168.9)
- added REF**: MountingHole_2.4mm, MountingHole:MountingHole_2.5mm, F.Cu at (85.0, 102.3)
- added REF**: MountingHole_2.5mm, MountingHole:MountingHole_2.5mm, F.Cu at (102.1, 71.8)
- added REF**: MountingHole_2.5mm, MountingHole:MountingHole_2.5mm, F.Cu at (152.7, 157.0)
- added microphone1: i2s INMP441, TerminalBlock:TerminalBlock_MaiXu_MX126-5.0-06P_1x06_P5.00mm, F.Cu at (43.5, 122.4)
- J1: value Conn_02x20_Counter_Clockwise -> radxa
- OLED1: footprint Connector_PinHeader_2.54mm:PinHeader_1x04_P2.54mm_Vertical -> TerminalBlock:TerminalBlock_MaiXu_MX126-5.0-04P_1x04_P5.00mm
- moved BNO055 84.4 mm to (84.7, 88.6)
- moved J1 8.89 mm to (133.6, 74.6)
- moved OLED1 7.29 mm to (45.6, 86.8), turned to 90 degrees
Connections:
- BNO055 pad 1: Net-(BNO055-Pin_1) -> +3V3
- BNO055 pad 4: Net-(BNO055-Pin_4) -> GND
- J1 pad 1: unconnected-(J1-Pin_1-Pad1) -> +3V3
- J1 pad 10: Net-(J1-Pin_10) -> unconnected-(J1-Pin_10-Pad10)
- J1 pad 11: Net-(J1-Pin_11) -> unconnected-(J1-Pin_11-Pad11)
- J1 pad 14: unconnected-(J1-Pin_14-Pad14) -> GND
- J1 pad 15: Net-(J1-Pin_10) -> unconnected-(J1-Pin_15-Pad15)
- J1 pad 16: Net-(J1-Pin_10) -> unconnected-(J1-Pin_16-Pad16)
- J1 pad 17: Net-(J1-Pin_10) -> unconnected-(J1-Pin_17-Pad17)
- J1 pad 18: Net-(J1-Pin_10) -> unconnected-(J1-Pin_18-Pad18)
- J1 pad 19: Net-(J1-Pin_10) -> unconnected-(J1-Pin_19-Pad19)
- J1 pad 2: unconnected-(J1-Pin_2-Pad2) -> +5V
- J1 pad 20: Net-(J1-Pin_10) -> GND
- J1 pad 21: Net-(J1-Pin_10) -> unconnected-(J1-Pin_21-Pad21)
- J1 pad 23: Net-(J1-Pin_10) -> unconnected-(J1-Pin_23-Pad23)
- J1 pad 24: Net-(J1-Pin_10) -> unconnected-(J1-Pin_24-Pad24)
- J1 pad 25: Net-(J1-Pin_10) -> GND
- J1 pad 26: Net-(J1-Pin_26) -> unconnected-(J1-Pin_26-Pad26)
- J1 pad 29: Net-(BNO055-Pin_1) -> unconnected-(J1-Pin_29-Pad29)
- J1 pad 30: Net-(J1-Pin_30) -> GND
- J1 pad 31: Net-(J1-Pin_31) -> unconnected-(J1-Pin_31-Pad31)
- J1 pad 32: Net-(J1-Pin_32) -> unconnected-(J1-Pin_32-Pad32)
- J1 pad 34: Net-(BNO055-Pin_2) -> GND
- J1 pad 37: Net-(J1-Pin_37) -> unconnected-(J1-Pin_37-Pad37)
- J1 pad 38: unconnected-(J1-Pin_38-Pad38) -> Net-(J1-Pin_38)
- J1 pad 39: unconnected-(J1-Pin_39-Pad39) -> GND
- J1 pad 4: Net-(J1-Pin_37) -> +5V
- J1 pad 40: unconnected-(J1-Pin_40-Pad40) -> Net-(J1-Pin_40)
- J1 pad 6: Net-(J1-Pin_10) -> GND
- J1 pad 7: Net-(J1-Pin_10) -> Net-(J1-Pin_7)
- J1 pad 8: Net-(J1-Pin_10) -> unconnected-(J1-Pin_8-Pad8)
- J1 pad 9: Net-(J1-Pin_9) -> GND
- OLED1 pad 1: Net-(BNO055-Pin_1) -> +3V3
- OLED1 pad 2: Net-(BNO055-Pin_2) -> GND
Routing:
- net +3V3: track 0.00 -> 420.6 mm
- net Net-(J1-Pin_35): track 0.00 -> 239.5 mm, vias 0 -> 3
- net Net-(J1-Pin_33): track 0.00 -> 148.7 mm, vias 0 -> 2
- net Net-(J1-Pin_38): track 0.00 -> 129.4 mm, vias 0 -> 2
- net Net-(J1-Pin_12): track 0.00 -> 122.0 mm, vias 0 -> 3
- net +5V: track 0.00 -> 120.4 mm, vias 0 -> 2
- net Net-(J3-Pin_12): track 0.00 -> 106.4 mm, vias 0 -> 2
- net Net-(J3-Pin_11): track 0.00 -> 93.6 mm
- net Net-(J1-Pin_27): track 0.00 -> 79.0 mm
- net Net-(J1-Pin_40): track 0.00 -> 70.7 mm, vias 0 -> 2
- net Net-(BNO055-Pin_2): track 0.00 -> 57.4 mm
- net Net-(BNO055-Pin_3): track 0.00 -> 51.3 mm
- net Net-(J1-Pin_28): track 0.00 -> 49.7 mm
- net Net-(J1-Pin_7): track 0.00 -> 47.1 mm
- added copper zone on B.Cu, net GND
Other:
- board size 248.7 x 150.6 mm -> 167 x 150 mm
- board text added: "+5V pin 2"
- board text added: "+5v pin 2"
- board text added: "+5v pin 4"
- board text added: "3.3v pin 1"
- board text added: "5V"
- board text added: "5V buck"
- board text added: "5V pin 4"
- board text added: "BCLK"
- board text added: "BNO055 RX et TX = scl et sda (soudage a faire)"
- board text added: "D E L O"
- board text added: "DIN"
- board text added: "DIN I2S3_SDO_M0 pin 40"
- board text added: "G"
- board text added: "GND"
- board text added: "GND BUCK"
- board text added: "GO BEYONDDDD PLUSS ULTRAA"
- board text added: "I2S3_LRCK_M0 pin 35"
- board text added: "I2S3_SCLK_M0 pin 12"
- board text added: "I2S3_SDI_M0 pin 38"
- board text added: "L/R"
- board text added: "MICROPHONE"
- board text added: "NONE"
- board text added: "SCK"
- board text added: "SCL"
- board text added: "SD"
- board text added: "SDA"
- board text added: "SDA pin 27"
- board text added: "UART5_RX_M1 pin 33"
- board text added: "VCC"
- board text added: "WS"
- board text added: "but nessie will live one day"
- board text added: "gnd"
- board text added: "gnd pin 14"
- board text added: "gnd pin 20"
- board text added: "gnd pin 25"
- board text added: "gnd pin 30"
- board text added: "gnd pin 34"
- board text added: "gnd pin 6"
- board text added: "gnd pin 9"
- board text added: "gnd pin9"
- board text added: "l/r"
- board text added: "lidar_tx"
- board text added: "made after hours of surfering"
- board text added: "none"
- board text added: "none pin 26"
- board text added: "none pin 29"
- board text added: "none pin 31"
- board text added: "none pin 32"
- board text added: "none pin 36"
- board text added: "ol sda"
- board text added: "oled scl"
- board text added: "p.s: i'm .... ALL MIGHT"
- board text added: "pin 14 gnd"
- board text added: "pin 20 gnd"
- board text added: "pin 25 gnd"
- board text added: "pin 34 gnd"
- board text added: "pin 37 none"
- board text added: "pin 39 gnd"
- board text added: "pin 40 gnd"
- board text added: "pwm sg90 motor pin 7"
- board text added: "radxa"
- board text added: "scl"
- board text added: "scl pin 28"
- board text added: "scl stab"
- board text added: "sda"
- board text added: "sda stab"
- board text added: "sg90 motor pmw pin 7"
- board text added: "sg90 pmw"
- board text added: "vcc"
- board text added: "vin pin 1"
- board text added: "ws"
- board text removed: "1"
- board text removed: "4"
- board text removed: "ZER0 3W_V1.11"
